File: synthmate_L432/_autosave-synthmate_L432.kicad_sch (KiCad schematic)
At the start: 45 parts, among them J1 USB_C_synthmate, J2 DIN-5_180degree, J3 USB_C_connector_board, J4 DIN-5_180degree, J5 Conn_01x16, J6 Conn_01x13, J7 Conn_01x04, J8 Conn_ST_STDC14, SW1 RotaryEncoder_Switch, SW2 SW_Push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

Commit message: fur hynek
Parts:
- J8: footprint (none) -> Samtec_LSHM-107-xx.x-x-DV-N
Changed lines of the file:
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@@
 			)
 		)
-		(property "Footprint" ""
+		(property "Footprint" "Samtec_LSHM-107-xx.x-x-DV-N"
 			(at 185.42 165.1 0)
 			(effects
