File: synthmate_L432/synthmate_L432.kicad_sch (KiCad schematic)
At the start: 45 parts, among them J1 USB_C_synthmate, J2 DIN-5_180degree, J3 USB_C_connector_board, J4 DIN-5_180degree, J5 Conn_01x16, J6 Conn_01x13, J7 Conn_01x04, J8 Conn_ST_STDC14, SW1 RotaryEncoder_Switch, SW2 SW_Push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

Commit message: 74LV14 / TPD4E02B04DQA
changed schmitt to 74LV14 and ESD to TPD4E02B04DQA
Parts:
- removed U5: 40106, Package_SO:TSSOP-14_4.4x5mm_P0.65mm, symbol 4xxx:40106
- added U5: TPD4E02B04DQA, Package_SON:USON-10_2.5x1.0mm_P0.5mm, symbol Power_Protection:TPD4E02B04DQA
- added U6: 74LV14, Package_DFN_QFN:Texas_S-PVQFN-N14, symbol 74xx:74LV14
- J8: footprint (none) -> Connector_PinHeader_1.27mm:PinHeader_2x07_P1.27mm_Vertical_SMD
- SW1: footprint Rotary_Encoder:RotaryEncoder_Bourns_Vertical_PEC12R-3x17F-Sxxxx -> Rotary_Encoder:RotaryEncoder_Alps_EC11E-Switch_Vertical_H20mm
- U2, U4: footprint Package_TO_SOT_SMD:SOT-23-6 -> (none)
Connections:
- net 3V3: now also J8.3 (VCC), U6.14 (3.3V); no longer U4.5 (VBUS)
- net 5V: no longer U2.5 (VBUS)
- net BOOT0: now also U6.6
- net GND: now also J8.5 (GND), J8.7 (GND), U5.3 (G), U5.8 (G), U6.13, U6.7 (GND); no longer U2.2 (GND), U4.2 (GND)
- net LPUART_RX: now also J1.B8 (SBU2), U5.5 (IO4); no longer U4.4 (I/O2)
- net LPUART_TX: now also J1.A8 (SBU1), U5.4 (IO3); no longer U4.6 (I/O1)
- net NRST: now also J8.12 (~{RST})
- net PA13: no longer U1.23 (PA13)
- net PA14: no longer U1.24 (PA14)
- net enc_A: now also U6.2
- net enc_B: now also U6.4
- net pushbutton_A: now also U6.8
- net pushbutton_B: now also U6.10
- net usb+: now also J1.A6 (D+), J1.B6 (D+), U5.2 (IO2); no longer U2.4 (I/O2)
- net usb-: now also J1.A7 (D-), J1.B7 (D-), U5.1 (IO1); no longer U2.6 (I/O1)
- net at U4.1 (I/O1): no longer J1.A8 (SBU1)
- net at U4.3 (I/O2): no longer J1.B8 (SBU2)
- net at C9.1, R13.2: now also U6.11
- net at C10.1, R14.1: now also U6.5
- net at C8.1, R12.2: now also U6.9
- net at C7.1, R9.1: now also U6.3
- net at C6.1, R8.1: now also U6.1
- net SWDIO: now reaches J8.4 (JTMS/SWDIO)
- net SWDIO: now also U1.23 (PA13)
- net SWCLK: now reaches J8.6 (JCLK/SWCLK)
- net SWCLK: now also U1.24 (PA14)
- removed net usb_N: J1.A7 (D-), J1.B7 (D-), U2.1 (I/O1)
- removed net usb_P: J1.A6 (D+), J1.B6 (D+), U2.3 (I/O2)
Other:
- note added: "Package_TO_SOT_SMD:SOT-23-6"
- note removed: "is in necessary to use pullup resistors when the overall current will note exceed 5mA?"
- note removed: "really not sure about BOOT0 and NRST"
- moved on the sheet: U2, U4
