File: synthmate_hyna_L432/synthmate_L432.kicad_sch (KiCad schematic)
At the start: 44 parts, among them J1 USB_C_synthmate, J2 DIN-5_180degree, J3 USB_C_connector_board, J4 DIN-5_180degree, J5 Conn_01x15, J7 Conn_01x04, J8 Conn_ST_STDC14, SW1 RotaryEncoder_Switch, SW2 SW_Push, SW3 SW_Push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

Commit message: added analog mux on main board nd adapter board
Parts:
- removed J7: Conn_01x04, Connector_PinSocket_2.54mm:PinSocket_1x04_P2.54mm_Vertical, symbol Connector_Generic:Conn_01x04
- removed U5: TPD4E02B04DQA, Package_SON:USON-10_2.5x1.0mm_P0.5mm, symbol Power_Protection:TPD4E02B04DQA
- added C15: 1uF, Capacitor_SMD:C_0603_1608Metric_Pad1.08x0.95mm_HandSolder, symbol Device:C_Polarized
- added D3, D4: BAT54J, Diode_SMD:D_SOD-323F, symbol Diode:BAT54J
- added J6: Conn_01x06, symbol Connector_Generic:Conn_01x06
- added R15: 2k4, Resistor_SMD:R_0603_1608Metric_Pad0.98x0.95mm_HandSolder, symbol Device:R
- added R16, R17, R18, R19: 220R, Resistor_SMD:R_0603_1608Metric_Pad0.98x0.95mm_HandSolder, symbol Device:R
- added SW4: SW_Slide_DPDT, symbol Switch:SW_Slide_DPDT
- added U2: TS3USB221ARSER, footprints:RSE10, symbol 2025-07-31_14-13-11:TS3USB221ARSER
- added U4: TS5A23159RSE, Package_DFN_QFN:Texas_R-PUQFN-N10, symbol Analog_Switch:TS5A23159RSE
Connections:
- net 3V3: now also C15.1, D3.1 (K), D4.1 (K), U2.10 (VCC)
- net 5V: now also R16.2
- net BOOT0: now also U2.9 (S)
- net GND: now also C15.2, R17.1, R19.1, U2.5 (GND), U2.6 (*OE)
- net LPUART_RX: now also D3.2 (A), U2.2 (1D-); no longer J1.B8 (SBU2)
- net LPUART_TX: now also R16.1, R17.2, U2.1 (1D+); no longer J1.A8 (SBU1)
- net adaptor_5V: now also J6.2 (Pin_2), J6.5 (Pin_5), R15.1, R18.2, U4.8 (VCC)
- net adaptor_GND: now also J6.1 (Pin_1), J6.6 (Pin_6), U4.3 (GND)
- net adaptor_LPUART_RX: now also J6.3 (Pin_3), U4.4, U4.9; no longer J3.A8 (SBU1)
- net adaptor_LPUART_TX: now also J6.4 (Pin_4), U4.2, U4.7; no longer J3.B8 (SBU2)
- net at J3.A5 (CC1): now also R15.2
- net at J3.A6 (D+): now also J3.B6 (D+), R18.1, R19.2, U4.6
- net at J3.A7 (D-): now also J3.B7 (D-), D4.2 (A), U4.10
- net USB_DN renamed usb_N
- net usb_N: now also U2.7 (D-); no longer U1.21 (PA11)
- net USB_DP renamed usb_P
- net usb_P: now also U2.8 (D+); no longer U1.22 (PA12)
- new net usb_mcu_N: U1.21 (PA11), U2.4 (2D-)
- new net usb_mcu_P: U1.22 (PA12), U2.3 (2D+)
- no-connect marks 10 -> 6
Other:
- note added: "Prevents voltage from exceeding ~3.3 V + Vf (~3.6 V)"
- note added: "TX is configured as open-drain output When LOW → sinks current → drives MIDI signal When HIGH (open) → current loop sees +5 V Safe. No level shifter needed. Works with 3.3 V MCU and 5 V current loop"
- note added: "need permanent logic 1 for usb operation"
- note added: "put 5V to CC1/CC1 to detect adaptor board connected and switch mux to uart operation?"
- note removed: "ToDo: Dat diode spravne pouzdro"
- note removed: "alternative TPS7A02 which CAPS?"
- note removed: "swappable TX RX pins"
- moved on the sheet: D1, J1, J3, R2, R3, R4

Commit message: cleanup
Parts:
- removed D3: BAT54J, Diode_SMD:D_SOD-323F, symbol Diode:BAT54J
- removed R16, R17: 220R, Resistor_SMD:R_0603_1608Metric_Pad0.98x0.95mm_HandSolder, symbol Device:R

Commit message: adapter board rx/tx switching logic
Parts:
- added U5: SN74LVC1G14DBV, Package_TO_SOT_SMD:SOT-23-5, symbol 74xGxx:SN74LVC1G14DBV
Connections:
- net adaptor_5V: now also U4.1, U4.5, U5.2, U5.4, U5.5 (VCC)
- net adaptor_GND: now also U5.3 (GND)
Other:
- note added: "LARGE VIAS"
- note added: "The MIC5365 has a typical soft-start time of ~1000–2000 µs (1–2 ms) depending on load and cap size. ➡️ Faster alternatives: MIC5219-3.3: similar footprint, faster transient response AP2112K-3.3: very common, fast startup, stable with 1–10 µF TLV75533P (TI): fast startup, very low dropout, great for MCUs"
- moved on the sheet: C13, J6, J8, SW4, U4C, U6F, U6G

Commit message: cleanup
Connections:
- net GND: now also SW3.2; no longer SW3.1
- net at R11.1, R13.1: now also SW3.1; no longer SW3.2
Changed lines of the file:
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@@
 		(lib_id "Switch:SW_Push")
 		(at 26.67 99.06 0)
+		(mirror y)
 		(unit 1)
 		(exclude_from_sim no)
@@
 		(on_board yes)
 		(dnp no)
-		(fields_autoplaced yes)
 		(property "Reference" "SW3"
 			(at 26.67 91.44 0)
