File: synthmate_hyna_L432/synthmate_L432.kicad_sch (KiCad schematic)
At the start: 51 parts, among them J1 USB_C_synthmate, J2 DIN-5_180degree, J3 USB_C_connector_board, J4 DIN-5_180degree, J5 Conn_01x15, J6 Conn_01x06, J8 Conn_ST_STDC14, SW1 RotaryEncoder_Switch, SW2 SW_Push, SW3 SW_Push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

Commit message: V2_gerber
Parts:
- removed J3: USB_C_connector_board, Connector_USB:USB_C_Receptacle_GCT_USB4105-xx-A_16P_TopMnt_Horizontal, symbol Connector:USB_C_Receptacle_USB2.0_16P
- removed J5: Conn_01x15, Connector_PinHeader_2.54mm:PinHeader_1x15_P2.54mm_Vertical, symbol Connector_Generic:Conn_01x15
- removed J6: Conn_01x06, symbol Connector_Generic:Conn_01x06
- removed R15: 2k4, Resistor_SMD:R_0603_1608Metric_Pad0.98x0.95mm_HandSolder, symbol Device:R
- removed R17: 470R, Resistor_SMD:R_0603_1608Metric_Pad0.98x0.95mm_HandSolder, symbol Device:R
- added H1, H2: MountingHole, MountingHole:MountingHole_2.1mm, symbol Mechanical:MountingHole
- added R18: 20k, Resistor_SMD:R_0603_1608Metric_Pad0.98x0.95mm_HandSolder, symbol Device:R
- added TP1, TP2, TP3, TP4, TP5, TP6: TestPoint, TestPoint:TestPoint_Pad_1.0x1.0mm, symbol Connector:TestPoint
- D3: footprint (none) -> Diode_SMD:D_0603_1608Metric
- SW2, SW3: footprint Button_Switch_THT:SW_TH_Tactile_Omron_B3F-10xx -> Button_Switch_THT:Marquardt_6450
Connections:
- net 3V3: now also R18.1
- net LPUART_RX: now also TP5.1
- net LPUART_TX: now also TP6.1
- net USART1_RX: now also U1.20 (PA10), TP2.1
- net at U1.19 (PA9), U4.2 (A): now also TP1.1
- net at J1.A5 (CC1), R2.2: no longer U2.9 (S)
- net PA15: no longer names the net of U1.25 (PA15)
- net PA15: now also TP3.1
- net PA7 renamed usb_switch
- net usb_switch: now also U2.9 (S), R18.2, TP4.1
- no-connect marks 6 -> 3
Other:
- note added: "midi 1.0 spec resistor, put there 0 ohm resistor"
- note removed: "DIN CONNECTORS JUST FOR ILLUSTRATION"
- note removed: "additional pins for debug"
- note removed: "midi 1.0 spec resistor"
- note removed: "put 5V to CC1/CC1 to detect adaptor board connected and switch mux to uart operation?"
- moved on the sheet: C15, D1, R4

Commit message: before autorouter, locked footprints and usb
Parts:
- removed H1, H2: MountingHole, MountingHole:MountingHole_2.1mm, symbol Mechanical:MountingHole
- removed SW2, SW3: SW_Push, Button_Switch_THT:Marquardt_6450, symbol Switch:SW_Push
- removed TP1, TP2, TP3, TP4, TP5, TP6: TestPoint, TestPoint:TestPoint_Pad_1.0x1.0mm, symbol Connector:TestPoint
- added C17, C18: 1uF, Capacitor_SMD:C_0603_1608Metric, symbol Device:C_Polarized
- added J3: Conn_01x02, Connector_PinHeader_1.00mm:PinHeader_1x02_P1.00mm_Vertical, symbol Connector_Generic:Conn_01x02
- added R15, R17: 10k, Resistor_SMD:R_0603_1608Metric, symbol Device:R
- added SW2, SW3, SW5: PB_86_A1, PB86:PB_86_A0, symbol PB_86_A1:PB_86_A1
- added U5: M95256-WMN6P, Package_SO:SOIC-8_3.9x4.9mm_P1.27mm, symbol Memory_EEPROM:M95256-WMN6P
- C10, C11, C12, C13, C15, C16, C2, C3, C4, C5, C6, C7, C8, C9: footprint Capacitor_SMD:C_0603_1608Metric_Pad1.08x0.95mm_HandSolder -> Capacitor_SMD:C_0603_1608Metric
- R1, R10, R11, R12, R13, R14, R16, R18, R2, R3, R4, R5, R6, R7, R8, R9: footprint Resistor_SMD:R_0603_1608Metric_Pad0.98x0.95mm_HandSolder -> Resistor_SMD:R_0603_1608Metric
- U3: value MIC5365-1.0YC5 -> MIC5365-3.3YC5
Connections:
- net LPUART_RX is gone; now on net usb_switch: U1.9 (PA3)
- net LPUART_TX is gone; now on net BOOT0: U1.8 (PA2)
- net PB3 is gone; now on net GND: U1.26 (PB3)
- net PB4 is gone; now on net GND: U1.27 (PB4)
- net PB5 is gone; now on net pushbutton_A: U1.28 (PB5)
- net PB6 is gone; now on net pushbutton_B: U1.29 (PB6)
- net 3V3: now also C18.1, R15.2, U5.7 (~{HOLD}), U5.8 (VCC)
- net BOOT0: no longer U1.10 (PA4)
- net GND: now also U1.18 (PA8), U1.2 (PC14), U1.3 (PC15), C17.2, C18.2, SW2.1 (B), SW3.1 (B), SW5.1 (B), U5.3 (~{W}), U5.4 (VSS); no longer U6.13
- net LED: now also U1.25 (PA15); no longer U1.18 (PA8)
- net pushbutton_A: now also U6.12; no longer U1.11 (PA5), U6.8
- net pushbutton_B: no longer U1.12 (PA6)
- net usb_switch: no longer U1.13 (PA7)
- net at R11.1, R13.1: now also SW2.2 (C)
- net at R10.1, R12.1: now also SW5.2 (C)
- net PB0: no longer names the net of U1.14 (PB0)
- net PB0: now also J3.2 (Pin_2)
- net PB1: no longer names the net of U1.15 (PB1)
- net PB1: now also J3.1 (Pin_1)
- net PB7 renamed pushbutton_C
- net pushbutton_C: now also U6.8
- new net: R15.1, R17.1, SW3.2 (C)
- new net: C17.1, R17.2, U6.13
- new net CS: U1.10 (PA4), U5.1 (~{S})
- new net MISO: U1.12 (PA6), U5.2 (Q)
- new net MOSI: U1.13 (PA7), U5.5 (D)
- new net SCK: U1.11 (PA5), U5.6 (C)
- no-connect marks 3 -> 0
Other:
- note added: "M95M04"
- note removed: "LARGE VIAS"
- moved on the sheet: C8, C9, J2, J4, J8, R10, R11, R12, R13, U6D, U6E, U6F

Commit message: naming cleanup
Parts:
- D2, D3: value D_Schottky -> 1N5819WS; footprint Diode_SMD:D_0603_1608Metric -> Diode_SMD:D_SOD-323
- J1: value USB_C_synthmate -> USB4105-GF-A-120
- U1: value STM32L432KCUx -> STM32L432KBU6
- U4: value SN74LV1T34DBV -> SN74LV1T34DBVR
- U5: value M95256-WMN6P -> M95M04-DRMN6TP
- U6: value 74LV14 -> SN74LV14APWR; footprint Package_DFN_QFN:Texas_S-PVQFN-N14 -> Package_SO:TSSOP-14_4.4x5mm_P0.65mm
Changed lines of the file:
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@@
 			)
 		)
-		(property "Value" "74LV14"
+		(property "Value" "SN74LV14APWR"
 			(at 160.02 43.18 0)
 			(effects
@@
 			)
 		)
-		(property "Footprint" "Package_DFN_QFN:Texas_S-PVQFN-N14"
+		(property "Footprint" "Package_SO:TSSOP-14_4.4x5mm_P0.65mm"
 			(at 160.02 49.53 0)
 			(effects
@@
 			)
 		)
-		(property "Value" "STM32L432KCUx"
+		(property "Value" "STM32L432KBU6"
 			(at 282.8133 123.19 0)
 			(effects
@@
 			)
 		)
-		(property "Value" "USB_C_synthmate"
+		(property "Value" "USB4105-GF-A-120"
 			(at 518.16 82.55 0)
 			(effects
@@
 			)
 		)
-		(property "Value" "74LV14"
+		(property "Value" "SN74LV14APWR"
 			(at 453.39 256.5399 0)
 			(effects
@@
 			)
 		)
-		(property "Footprint" "Package_DFN_QFN:Texas_S-PVQFN-N14"
+		(property "Footprint" "Package_SO:TSSOP-14_4.4x5mm_P0.65mm"
 			(at 447.04 255.27 0)
 			(effects
@@
 			)
 		)
-		(property "Value" "D_Schottky"
+		(property "Value" "1N5819WS"
 			(at 341.63 97.4724 90)
 			(effects
@@
 			)
 		)
-		(property "Footprint" "Diode_SMD:D_0603_1608Metric"
+		(property "Footprint" "Diode_SMD:D_SOD-323"
 			(at 339.09 96.52 0)
 			(effects
@@
 			)
 		)
-		(property "Description" "Schottky diode"
+		(property "Description" "1N5819WS"
 			(at 339.09 96.52 0)
 			(effects
@@
 			)
 		)
-		(property "Value" "74LV14"
+		(property "Value" "SN74LV14APWR"
 			(at 54.61 43.18 0)
 			(effects
@@
 			)
 		)
-		(property "Footprint" "Package_DFN_QFN:Texas_S-PVQFN-N14"
+		(property "Footprint" "Package_SO:TSSOP-14_4.4x5mm_P0.65mm"
 			(at 54.61 49.53 0)
 			(effects
@@
 			)
 		)
-		(property "Value" "D_Schottky"
+		(property "Value" "1N5819WS"
 			(at 255.27 172.4024 90)
 			(effects
@@
 			)
 		)
-		(property "Footprint" "Diode_SMD:D_0603_1608Metric"
+		(property "Footprint" "Diode_SMD:D_SOD-323"
 			(at 252.73 171.45 0)
 			(effects
@@
 			)
 		)
-		(property "Value" "74LV14"
+		(property "Value" "SN74LV14APWR"
 			(at 100.33 102.87 0)
 			(effects
@@
 			)
 		)
-		(property "Footprint" "Package_DFN_QFN:Texas_S-PVQFN-N14"
+		(property "Footprint" "Package_SO:TSSOP-14_4.4x5mm_P0.65mm"
 			(at 100.33 109.22 0)
 			(effects
@@
 			)
 		)
-		(property "Value" "M95256-WMN6P"
+		(property "Value" "M95M04-DRMN6TP"
 			(at 352.6633 128.27 0)
 			(effects
@@
 			)
 		)
-		(property "Value" "74LV14"
+		(property "Value" "SN74LV14APWR"
 			(at 160.02 69.85 0)
 			(effects
@@
 			)
 		)
-		(property "Footprint" "Package_DFN_QFN:Texas_S-PVQFN-N14"
+		(property "Footprint" "Package_SO:TSSOP-14_4.4x5mm_P0.65mm"
 			(at 160.02 76.2 0)
 			(effects
@@
 		(fields_autoplaced yes)
 		(property "Reference" "U4"
-			(at 344.17 69.7798 0)
+			(at 345.44 69.7798 0)
 			(effects
 				(font
@@
 			)
 		)
-		(property "Value" "SN74LV1T34DBV"
-			(at 344.17 72.3198 0)
+		(property "Value" "SN74LV1T34DBVR"
+			(at 345.44 72.3198 0)
 			(effects
 				(font
@@
 			)
 		)
-		(property "Value" "74LV14"
+		(property "Value" "SN74LV14APWR"
 			(at 100.33 139.7 0)
 			(effects
@@
 			)
 		)
-		(property "Footprint" "Package_DFN_QFN:Texas_S-PVQFN-N14"
+		(property "Footprint" "Package_SO:TSSOP-14_4.4x5mm_P0.65mm"
 			(at 100.33 146.05 0)
 			(effects
@@
 			)
 		)
-		(property "Value" "74LV14"
+		(property "Value" "SN74LV14APWR"
 			(at 100.33 184.15 0)
 			(effects
@@
 			)
 		)
-		(property "Footprint" "Package_DFN_QFN:Texas_S-PVQFN-N14"
+		(property "Footprint" "Package_SO:TSSOP-14_4.4x5mm_P0.65mm"
 			(at 100.33 190.5 0)
 			(effects

Commit message: 23_1
Parts:
- added J5: Conn_01x04, Connector_PinHeader_2.54mm:PinHeader_1x04_P2.54mm_Vertical, symbol Connector_Generic:Conn_01x04
- U3: value MIC5365-3.3YC5 -> MIC5365-3.3YC5-TR
Connections:
- net 3V3: now also U5.3 (~{W}), J5.4 (Pin_4)
- net GND: now also J5.1 (Pin_1); no longer U5.3 (~{W})
- net SWCLK: now also J5.2 (Pin_2)
- net SWDIO: now also J5.3 (Pin_3)
Changed lines of the file:
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@@
 	)
 	(junction
+		(at 334.01 135.89)
+		(diameter 0)
+		(color 0 0 0 0)
+	)
+	(junction
 		(at 22.86 148.59)
 		(diameter 0)
@@
 	(wire
 		(pts
+			(xy 334.01 135.89) (xy 340.36 135.89)
+		)
+		(stroke
+			(width 0)
+			(type default)
+		)
+	)
+	(wire
+		(pts
 			(xy 293.37 95.25) (xy 309.88 95.25)
 		)
@@
 	(wire
 		(pts
+			(xy 408.94 241.3) (xy 408.94 248.92)
+		)
+		(stroke
+			(width 0)
+			(type default)
+		)
+	)
+	(wire
+		(pts
 			(xy 474.98 100.33) (xy 474.98 107.95)
 		)
@@
 	(wire
 		(pts
+			(xy 402.59 241.3) (xy 408.94 241.3)
+		)
+		(stroke
+			(width 0)
+			(type default)
+		)
+	)
+	(wire
+		(pts
 			(xy 436.88 36.83) (xy 439.42 36.83)
 		)
@@
 	(wire
 		(pts
-			(xy 334.01 124.46) (xy 334.01 133.35)
-		)
-		(stroke
-			(width 0)
-			(type default)
-		)
-	)
-	(wire
-		(pts
 			(xy 293.37 97.79) (xy 317.5 97.79)
 		)
@@
 	(wire
 		(pts
+			(xy 334.01 133.35) (xy 334.01 135.89)
+		)
+		(stroke
+			(width 0)
+			(type default)
+		)
+	)
+	(wire
+		(pts
 			(xy 267.97 97.79) (xy 267.97 100.33)
 		)
@@
 	(wire
 		(pts
-			(xy 334.01 124.46) (xy 337.82 124.46)
-		)
-		(stroke
-			(width 0)
-			(type default)
-		)
-	)
-	(wire
-		(pts
 			(xy 518.16 130.81) (xy 518.16 125.73)
 		)
@@
 	(wire
 		(pts
-			(xy 322.58 135.89) (xy 340.36 135.89)
+			(xy 322.58 135.89) (xy 334.01 135.89)
 		)
 		(stroke
@@
 		)
 	)
+	(global_label "3V3"
+		(shape input)
+		(at 408.94 256.54 180)
+		(fields_autoplaced yes)
+		(effects
+			(font
+				(size 1.27 1.27)
+			)
+			(justify right)
+		)
+		(property "Intersheetrefs" "${INTERSHEET_REFS}"
+			(at 402.4472 256.54 0)
+			(effects
+				(font
+					(size 1.27 1.27)
+				)
+				(justify right)
+				(hide yes)
+			)
+		)
+	)
 	(global_label "NRST"
 		(shape input)
@@
 		)
 	)
+	(global_label "SWDIO"
+		(shape input)
+		(at 408.94 254 180)
+		(fields_autoplaced yes)
+		(effects
+			(font
+				(size 1.27 1.27)
+			)
+			(justify right)
+		)
+		(property "Intersheetrefs" "${INTERSHEET_REFS}"
+			(at 400.0886 254 0)
+			(effects
+				(font
+					(size 1.27 1.27)
+				)
+				(justify right)
+				(hide yes)
+			)
+		)
+	)
 	(global_label "LED"
 		(shape input)
@@
 		)
 	)
+	(global_label "SWCLK"
+		(shape input)
+		(at 408.94 251.46 180)
+		(fields_autoplaced yes)
+		(effects
+			(font
+				(size 1.27 1.27)
+			)
+			(justify right)
+		)
+		(property "Intersheetrefs" "${INTERSHEET_REFS}"
+			(at 399.7258 251.46 0)
+			(effects
+				(font
+					(size 1.27 1.27)
+				)
+				(justify right)
+				(hide yes)
+			)
+		)
+	)
 	(global_label "3V3"
 		(shape input)
@@
 	)
 	(symbol
+		(lib_id "Connector_Generic:Conn_01x04")
+		(at 414.02 251.46 0)
+		(unit 1)
+		(exclude_from_sim no)
+		(in_bom yes)
+		(on_board yes)
+		(dnp no)
+		(fields_autoplaced yes)
+		(property "Reference" "J5"
+			(at 416.56 251.4599 0)
+			(effects
+				(font
+					(size 1.27 1.27)
+				)
+				(justify left)
+			)
+		)
+		(property "Value" "Conn_01x04"
+			(at 416.56 253.9999 0)
+			(effects
+				(font
+					(size 1.27 1.27)
+				)
+				(justify left)
+			)
+		)
+		(property "Footprint" "Connector_PinHeader_2.54mm:PinHeader_1x04_P2.54mm_Vertical"
+			(at 414.02 251.46 0)
+			(effects
+				(font
+					(size 1.27 1.27)
+				)
+				(hide yes)
+			)
+		)
+		(property "Datasheet" "~"
+			(at 414.02 251.46 0)
+			(effects
+				(font
+					(size 1.27 1.27)
+				)
+				(hide yes)
+			)
+		)
+		(property "Description" "Generic connector, single row, 01x04, script generated (kicad-library-utils/schlib/autogen/connector/)"
+			(at 414.02 251.46 0)
+			(effects
+				(font
+					(size 1.27 1.27)
+				)
+				(hide yes)
+			)
+		)
+		(pin "1"
+		)
+		(pin "2"
+		)
+		(pin "3"
+		)
+		(pin "4"
+		)
+		(instances
+			(project ""
+				(path "/51b18779-52cf-4d77-bac0-6803e3c57cb1"
+					(reference "J5")
+					(unit 1)
+				)
+			)
+		)
+	)
+	(symbol
 		(lib_id "power:GND")
 		(at 90.17 153.67 0)
@@
 			)
 		)
-		(property "Value" "MIC5365-3.3YC5"
+		(property "Value" "MIC5365-3.3YC5-TR"
 			(at 309.88 162.56 0)
 			(effects
@@
 	)
 	(symbol
-		(lib_id "power:GND")
-		(at 337.82 124.46 0)
-		(unit 1)
-		(exclude_from_sim no)
-		(in_bom yes)
-		(on_board yes)
-		(dnp no)
-		(fields_autoplaced yes)
-		(property "Reference" "#PWR011"
-			(at 337.82 130.81 0)
-			(effects
-				(font
-					(size 1.27 1.27)
-				)
-				(hide yes)
-			)
-		)
-		(property "Value" "GND"
-			(at 337.82 129.54 0)
-			(effects
-				(font
-					(size 1.27 1.27)
-				)
-			)
-		)
-		(property "Footprint" ""
-			(at 337.82 124.46 0)
-			(effects
-				(font
-					(size 1.27 1.27)
-				)
-				(hide yes)
-			)
-		)
-		(property "Datasheet" ""
-			(at 337.82 124.46 0)
-			(effects
-				(font
-					(size 1.27 1.27)
-				)
-				(hide yes)
-			)
-		)
-		(property "Description" "Power symbol creates a global label with name \"GND\" , ground"
-			(at 337.82 124.46 0)
-			(effects
-				(font
-					(size 1.27 1.27)
-				)
-				(hide yes)
-			)
-		)
-		(pin "1"
-		)
-		(instances
-			(project "synthmate_L432"
-				(path "/51b18779-52cf-4d77-bac0-6803e3c57cb1"
-					(reference "#PWR011")
-					(unit 1)
-				)
-			)
-		)
-	)
-	(symbol
 		(lib_id "PB_86_A1:PB_86_A1")
 		(at 33.02 193.04 0)
@@
 				)
 			)
+		)
+	)
+	(symbol
+		(lib_id "power:GND")
+		(at 402.59 241.3 0)
+		(unit 1)
+		(exclude_from_sim no)
+		(in_bom yes)
+		(on_board yes)
+		(dnp no)
+		(fields_autoplaced yes)
+		(property "Reference" "#PWR011"
+			(at 402.59 247.65 0)
+			(effects
+				(font
+					(size 1.27 1.27)
+				)
+				(hide yes)
+			)
+		)
+		(property "Value" "GND"
+			(at 402.59 246.38 0)
+			(effects
+				(font
+					(size 1.27 1.27)
+				)
+			)
+		)
+		(property "Footprint" ""
+			(at 402.59 241.3 0)
+			(effects
+				(font
+					(size 1.27 1.27)
+				)
+				(hide yes)
+			)
+		)
+		(property "Datasheet" ""
+			(at 402.59 241.3 0)
+			(effects
+				(font
+					(size 1.27 1.27)
+				)
+				(hide yes)
+			)
+		)
+		(property "Description" "Power symbol creates a global label with name \"GND\" , ground"
+			(at 402.59 241.3 0)
+			(effects
+				(font
+					(size 1.27 1.27)
+				)
+				(hide yes)
+			)
+		)
+		(pin "1"
+		)
+		(instances
+			(project "synthmate_L432"
+				(path "/51b18779-52cf-4d77-bac0-6803e3c57cb1"
+					(reference "#PWR011")
+					(unit 1)
+				)
+			)
